File: SCHEMATICS/KiCad cycle tracker.kicad_sch (KiCad schematic)
At the start: 28 parts, among them Q1 Q_NMOS, Q2 Q_NMOS, SW1 SW_SPST, SW2 SW_Push, U1 ESP32-WROOM-32, U2 TP4056-42-ESOP8, U3 AP2112K-3.3, U4 MAX30205MTA_, U5 AHT20, U6 MAX30102, U7 MPU-6050-A, U8 DW01A

Commit message: updates correct schematic uploaded
Parts:
- removed C7: 0.1uF, symbol Device:C_US
- removed Q1, Q2: Q_NMOS, symbol Device:Q_NMOS
- removed R6: 100, symbol Device:R
- removed R7: 1k, symbol Device:R
- removed U1: ESP32-WROOM-32, RF_Module:ESP32-WROOM-32, symbol RF_Module:ESP32-WROOM-32
- removed U2: TP4056-42-ESOP8, Package_SO:SOIC-8-1EP_3.9x4.9mm_P1.27mm_EP2.41x3.3mm_ThermalVias, symbol Battery_Management:TP4056-42-ESOP8
- removed U8: DW01A, Package_TO_SOT_SMD:SOT-23-6, symbol Battery_Management:DW01A
- added U1: DEVKIT_V1_ESP32-WROOM-32, DEVKIT_V1_ESP32-WROOM-32:MODULE_DEVKIT_V1_ESP32-WROOM-32, symbol DEVKIT_V1_ESP32-WROOM-32:DEVKIT_V1_ESP32-WROOM-32
- C2: value 0,1uF -> 0.1uF
Connections:
- net 3V3: now also U1.1 (3V3)
- net GND: now also D1.1 (K), U1.14 (GND1), U1.32 (GND2), U1.38 (GND3); no longer D1.2 (A)
- net SCL: now also U1.36 (IO22)
- net SDA: now also U1.33 (IO21)
- net at BT1.1 (+), R3.2: no longer SW1.1 (A)
- net at SW2.1: now also U1.25 (IO0)
- net at R5.1: now also D1.2 (A); no longer D1.1 (K)
- net at R5.2: now also U1.24 (IO2)
- net at R3.1, R4.2: now also U1.5 (IO34)
- no-connect marks 43 -> 40
Other:
- note added: "B+"
- note added: "B-"
- note added: "OUT+"
- note added: "OUT-"
- note added: "TP4056 Protected Module"
- moved on the sheet: D1, R1, R2, R5, SW1, SW2

Commit message: Corrected schematics uploaded
Parts:
- removed D1: LED, symbol Device:LED
- removed R5: 220, symbol Device:R
- removed SW2: SW_Push, symbol Switch:SW_Push
Connections:
- no-connect marks 40 -> 42
